File: starter_board/starter_board.kicad_sch (KiCad schematic)
At the start: 42 parts, among them J1 Conn_01x10, J2 Conn_01x10, J3 ICSP, J4 USB_B_Micro, U1 ATmega32U4-A, Y1 16MHz

Commit message: update board files for A24
Other:
- title: IEEE - DIY LEDs -> Essentials of PCB Design Starter Board
