File: starter_board/starter_board.kicad_pcb (KiCad board)
At the start: 2 copper layers, 102 x 40 mm, 10 parts, among them J1 Conn_01x10, J2 Conn_01x10, J3 ICSP, J4 USB_B_Micro, U1 ATmega32U4-A, Y1 16MHz

Commit message: update board files for A24
Parts:
- removed the G*** at (126.0, 162.0)
Routing:
- net GND: vias 1 -> 0
Other:
- board text added: "WPI IEEE | A24"
- board text removed: "locked"

Commit message: lock components
Other:
- board text added: "JLCJLCJLCJLC"
Changed lines of the file:
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@@
 		(pad_to_mask_clearance 0)
 		(allow_soldermask_bridges_in_footprints no)
-		(grid_origin 82 135)
+		(grid_origin 48.006 165.292)
 		(pcbplotparams
 			(layerselection 0x00010fc_ffffffff)
@@
 	(net 39 "/D10")
 	(footprint "Capacitor_SMD:C_0805_2012Metric_Pad1.18x1.45mm_HandSolder"
+		(locked yes)
 		(layer "F.Cu")
 		(at 69.342 157.099 -90)
@@
 	)
 	(footprint "Crystal:Crystal_SMD_5032-2Pin_5.0x3.2mm"
+		(locked yes)
 		(layer "F.Cu")
 		(at 67.564 152.781 180)
@@
 	)
 	(footprint "LOGO"
-		(locked yes)
 		(layer "F.Cu")
 		(at 142.15 161.8)
@@
 	)
 	(footprint "Capacitor_SMD:C_0805_2012Metric_Pad1.18x1.45mm_HandSolder"
+		(locked yes)
 		(layer "F.Cu")
 		(at 65.532 157.099 -90)
@@
 		(start 48.006 125.292)
 		(end 150.006 165.292)
+		(locked yes)
 		(stroke
 			(width 0.1)
@@
 	)
 	(gr_text "WPI IEEE | A24"
-		(locked yes)
 		(at 78.1 151 90)
 		(layer "B.SilkS")
@@
 		)
 	)
+	(gr_text "JLCJLCJLCJLC"
+		(at 149.006 164.292 0)
+		(layer "B.SilkS")
+		(effects
+			(font
+				(size 0.8 0.8)
+				(thickness 0.15)
+				(bold yes)
+			)
+			(justify left bottom mirror)
+		)
+	)
 	(gr_text "."
+		(locked yes)
 		(at 59.45 152.25 0)
 		(layer "F.SilkS")
@@
 	)
 	(gr_text "8"
+		(locked yes)
 		(at 67.5 165.25 0)
 		(layer "F.SilkS")
@@
 	)
 	(gr_text "1"
+		(locked yes)
 		(at 57.4 165.25 0)
 		(layer "F.SilkS")
@@
 	)
 	(gr_text "13"
+		(locked yes)
 		(at 72.15 126.6 0)
 		(layer "F.SilkS")
@@
 	)
 	(gr_text "A3"
+		(locked yes)
 		(at 62 126.6 0)
 		(layer "F.SilkS")
@@
 	)
 	(gr_text "A2"
+		(locked yes)
 		(at 64.6 126.6 0)
 		(layer "F.SilkS")
@@
 	)
 	(gr_text "9"
+		(locked yes)
 		(at 70 165.25 0)
 		(layer "F.SilkS")
@@
 	)
 	(gr_text "A5"
+		(locked yes)
 		(at 56.95 126.6 0)
 		(layer "F.SilkS")
@@
 	)
 	(gr_text "AR"
+		(locked yes)
 		(at 51.9 126.6 0)
 		(layer "F.SilkS")
@@
 	)
 	(gr_text "3"
+		(locked yes)
 		(at 52.2 165.25 0)
 		(layer "F.SilkS")
@@
 	)
 	(gr_text "4"
+		(locked yes)
 		(at 64.9 165.25 0)
 		(layer "F.SilkS")
@@
 	)
 	(gr_text "5V"
+		(locked yes)
 		(at 49.2 126.6 0)
 		(layer "F.SilkS")
@@
 	)
 	(gr_text "A0"
+		(locked yes)
 		(at 69.7 126.6 0)
 		(layer "F.SilkS")
@@
 	)
 	(gr_text "G"
+		(locked yes)
 		(at 54.75 126.6 0)
 		(layer "F.SilkS")
@@
 	)
 	(gr_text "A4"
+		(locked yes)
 		(at 59.45 126.6 0)
 		(layer "F.SilkS")
@@
 	)
 	(gr_text "A1"
+		(locked yes)
 		(at 67.2 126.6 0)
 		(layer "F.SilkS")
@@
 	)
 	(gr_text "G"
+		(locked yes)
 		(at 49.6 165.25 0)
 		(layer "F.SilkS")
@@
 	)
 	(gr_text "10"
+		(locked yes)
 		(at 72.2 165.25 0)
 		(layer "F.SilkS")
@@
 	)
 	(gr_text "0"
+		(locked yes)
 		(at 59.9 165.25 0)
 		(layer "F.SilkS")
@@
 	)
 	(gr_text "2"
+		(locked yes)
 		(at 54.8 165.25 0)
 		(layer "F.SilkS")
@@
 	)
 	(gr_text "11"
+		(locked yes)
 		(at 62.05 165.25 0)
 		(layer "F.SilkS")
@@
 		(end 69.342 156.0615)
 		(width 0.25)
+		(locked yes)
 		(layer "F.Cu")
 		(net 3)
@@
 		(end 69.414 152.781)
 		(width 0.25)
+		(locked yes)
 		(layer "F.Cu")
 		(net 3)
@@
 		(end 67.96 151.327)
 		(width 0.25)
+		(locked yes)
 		(layer "F.Cu")
 		(net 3)
@@
 		(end 69.414 155.9895)
 		(width 0.25)
+		(locked yes)
 		(layer "F.Cu")
 		(net 3)
@@
 		(end 65.714 155.8795)
 		(width 0.25)
+		(locked yes)
 		(layer "F.Cu")
 		(net 4)
@@
 		(end 65.532 156.0615)
 		(width 0.25)
+		(locked yes)
 		(layer "F.Cu")
 		(net 4)
@@
 		(end 67.16 151.335)
 		(width 0.25)
+		(locked yes)
 		(layer "F.Cu")
 		(net 4)
@@
 		(end 65.714 152.781)
 		(width 0.25)
+		(locked yes)
 		(layer "F.Cu")
 		(net 4)
 	)
 	(segment
-		(start 62.2 154.8)
-		(end 62.4 154.8)
-		(width 0.25)
-		(layer "B.Cu")
-		(net 34)
-	)
-	(segment

Commit message: Add updated term to board
Other:
- board text added: "WPI IEEE | A25"
- board text removed: "WPI IEEE | A24"
Changed lines of the file:
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@@
 		(layer "Edge.Cuts")
 	)
-	(gr_text "WPI IEEE | A24"
+	(gr_text "WPI IEEE | A25"
 		(at 78.1 151 90)
 		(layer "B.SilkS")

Commit message: Update starter board for KiCad 9.0.7
Other:
- board text added: "pcb.wpi.edu"
- board text removed: "WPI IEEE | A25"
